File: boostier.kicad_sch (KiCad schematic)
At the start: 7 parts, among them U1 TLV61070ADBV, U2 SN74LVC1G125DBV

Commit message: Minor cleanup.
Connections:
- net BOOST_EN renamed 5V_EN
- net LED_DATA_3V3 renamed LED_D3V
- net LED_DATA_5V renamed LED_D5V
- net V_OUT renamed 5V
Changed lines of the file:
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@@
 		)
 	)
-	(global_label "BOOST_EN"
+	(global_label "5V_EN"
 		(shape input)
 		(at 128.27 114.3 180)
@@
 		)
 		(property "Intersheetrefs" "${INTERSHEET_REFS}"
-			(at 115.7296 114.3 0)
+			(at 119.5396 114.3 0)
 			(effects
 				(font
@@
 		)
 	)
-	(global_label "LED_DATA_3V3"
+	(global_label "LED_D3V"
 		(shape input)
 		(at 193.04 100.33 0)
@@
 		)
 		(property "Intersheetrefs" "${INTERSHEET_REFS}"
-			(at 209.3299 100.33 0)
+			(at 204.008 100.33 0)
 			(effects
 				(font
@@
 		)
 	)
-	(global_label "BOOST_EN"
+	(global_label "5V_EN"
 		(shape input)
 		(at 182.88 85.09 180)
@@
 		)
 		(property "Intersheetrefs" "${INTERSHEET_REFS}"
-			(at 170.3396 85.09 0)
+			(at 174.1496 85.09 0)
 			(effects
 				(font
@@
 		)
 	)
-	(global_label "V_OUT"
+	(global_label "5V"
 		(shape input)
 		(at 189.23 111.76 0)
@@
 		)
 		(property "Intersheetrefs" "${INTERSHEET_REFS}"
-			(at 197.9 111.76 0)
+			(at 194.5133 111.76 0)
 			(effects
 				(font
@@
 		)
 	)
-	(global_label "LED_DATA_5V"
+	(global_label "LED_D5V"
 		(shape input)
 		(at 193.04 72.39 0)
@@
 		)
 		(property "Intersheetrefs" "${INTERSHEET_REFS}"
-			(at 208.1204 72.39 0)
+			(at 204.008 72.39 0)
 			(effects
 				(font

Commit message: Cleanup schematic/PCB mismatching net names
Parts:
- U2: value SN74LVC1G125DBV -> SN74LV1T126DBVR
Connections:
- net BOOST_SW: now reaches L1.2, U1.1 (SW)
- net BOOST_FB: now reaches R1.2, R2.1, U1.4 (V_{FB})
Changed lines of the file:
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@@
+		)
+	)
+	(global_label "BOOST_SW"
+		(shape input)
+		(at 162.56 109.22 0)
+		(fields_autoplaced yes)
+		(effects
+			(font
+				(size 1.27 1.27)
+			)
+			(justify left)
+		)
+		(property "Intersheetrefs" "${INTERSHEET_REFS}"
+			(at 175.2818 109.22 0)
+			(effects
+				(font
+					(size 1.27 1.27)
+				)
+				(justify left)
+				(hide yes)
+			)
 		)
 	)
@@
 				)
 				(justify right)
+				(hide yes)
+			)
+		)
+	)
+	(global_label "BOOST_FB"
+		(shape input)
+		(at 168.91 119.38 0)
+		(fields_autoplaced yes)
+		(effects
+			(font
+				(size 1.27 1.27)
+			)
+			(justify left)
+		)
+		(property "Intersheetrefs" "${INTERSHEET_REFS}"
+			(at 181.3295 119.38 0)
+			(effects
+				(font
+					(size 1.27 1.27)
+				)
+				(justify left)
 				(hide yes)
 			)
@@
 			)
 		)
-		(property "Value" "SN74LVC1G125DBV"
+		(property "Value" "SN74LV1T126DBVR"
 			(at 209.55 87.2646 90)
 			(effects
